File: PA/PA.kicad_pcb (KiCad board)
At the start: 2 copper layers, 100 x 100 mm, 126 parts, among them J1 Conn_Coaxial, J10 Conn_01x01, J11 Conn_01x01, J12 Conn_01x01, J13 Conn_01x01, J14 Conn_01x01, J15 Conn_01x01, J16 Conn_01x01, J17 Conn_01x01, J18 Conn_01x01, J19 Conn_01x01, J2 Conn_01x02, J20 Conn_01x01, J21 Conn_01x01, J22 Conn_01x01, J23 Conn_01x01, J24 Conn_01x01, J25 Conn_01x01, J26 Conn_01x01, J27 Conn_01x01, J28 Conn_01x01, J3 Conn_Coaxial, J4 Conn_01x02, J5 Conn_01x02, J6 Conn_01x01, J7 Conn_01x01, J8 Conn_01x01, J9 Conn_01x01, Q1 2N3904, Q2 IRF510N, Q3 IRF510N, Q4 2N3906, Q5 IRF510N, Q6 2N3904, T1 Transformer_1P1Sdotted, T2 Transformer_1P1Sdotted, T3 Transformer_1P1Sdotted

Commit message: Tightened up components
Parts:
- C4: value 1 nF -> 10 nF
- R10, R6, R7, R8: footprint Resistors_THT:R_Axial_DIN0411_L9.9mm_D3.6mm_P12.70mm_Horizontal -> Resistors_THT:R_Axial_DIN0207_L6.3mm_D2.5mm_P10.16mm_Horizontal
- moved C14 22.1 mm to (126.8, 44.4), turned to 180 degrees
- moved C13 20.0 mm to (97.4, 44.6), turned to 180 degrees
- moved C16 17.6 mm to (92.5, 52.5)
- moved C10 14.0 mm to (128.2, 53.4), turned to 270 degrees
- moved C19 12.9 mm to (107.7, 56.6), turned to 0 degrees
- moved D9 12.5 mm to (115.5, 58.4), turned to 270 degrees
- moved D8 11.8 mm to (81.8, 58.1)
- moved C11 11.3 mm to (96.8, 47.8), turned to 180 degrees
- moved D4 11.0 mm to (109.5, 89.6)
- moved C1 10.8 mm to (98.1, 92.7)
- moved C12 10.6 mm to (123.6, 47.9), turned to 180 degrees
- moved RLY1 10.6 mm to (103.4, 86.0)
- moved C15 10.3 mm to (101.0, 95.9)
- moved T3 10.1 mm to (99.9, 69.2)
- moved C5 9.65 mm to (68.8, 55.9), turned to 0 degrees
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Routing:
- net Net-(C1-Pad1): track 100.1 -> 82.6 mm
- net Net-(D3-Pad2): track 12.1 -> 28.8 mm
- net AMPINPUT: track 40.3 -> 24.7 mm
- net Net-(JP5-Pad2): track 7.95 -> 19.5 mm
- net Net-(C11-Pad1): track 53.4 -> 63.5 mm
- net Net-(JP6-Pad2): track 15.4 -> 23.8 mm
- net PASUPPLY: track 131.2 -> 139.3 mm
- net Net-(J3-Pad1): track 57.5 -> 49.4 mm
- net Net-(C5-Pad2): track 2.94 -> 9.74 mm
- net Net-(C6-Pad1): track 10.7 -> 17.3 mm
- net Net-(C10-Pad1): track 18.6 -> 13.6 mm
- net Net-(C12-Pad1): track 47.5 -> 52.5 mm
- net Net-(D10-Pad1): track 2.90 -> 7.32 mm
- net Net-(C2-Pad1): track 30.5 -> 26.7 mm
- net Net-(L2-Pad1): track 19.7 -> 16.6 mm
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