File: PA/Filters.sch (KiCad schematic (older format))
At the start: 42 parts, among them J10 Conn_01x01, J11 Conn_01x01, J12 Conn_01x01, J13 Conn_01x01, J14 Conn_01x01, J15 Conn_01x01, J16 Conn_01x01, J17 Conn_01x01, J18 Conn_01x01, J19 Conn_01x01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

Commit message: Made filter capacitors mica or 1206 SMT
Parts:
- C23, C24, C25, C26, C27, C28, C29, C30, C31, C32, C33, C34, C35, C36, C37: footprint Capacitors_THT:C_Disc_D7.5mm_W5.0mm_P7.50mm -> PA:C_Disc_SMD
Changed lines of the file:
@@
 F 0 "C23" H 2510 1970 50  0000 L CNN
 F 1 "C_Small" H 2510 1820 50  0000 L CNN
-F 2 "Capacitors_THT:C_Disc_D7.5mm_W5.0mm_P7.50mm" H 2500 1900 50  0001 C CNN
+F 2 "PA:C_Disc_SMD" H 2500 1900 50  0001 C CNN
 F 3 "" H 2500 1900 50  0001 C CNN
 	1    2500 1900
@@
 F 0 "C24" H 3060 2020 50  0000 L CNN
 F 1 "C_Small" H 3060 1870 50  0000 L CNN
-F 2 "Capacitors_THT:C_Disc_D7.5mm_W5.0mm_P7.50mm" H 3050 1950 50  0001 C CNN
+F 2 "PA:C_Disc_SMD" H 3050 1950 50  0001 C CNN
 F 3 "" H 3050 1950 50  0001 C CNN
 	1    3050 1950
@@
 F 0 "C25" H 3660 2020 50  0000 L CNN
 F 1 "C_Small" H 3660 1870 50  0000 L CNN
-F 2 "Capacitors_THT:C_Disc_D7.5mm_W5.0mm_P7.50mm" H 3650 1950 50  0001 C CNN
+F 2 "PA:C_Disc_SMD" H 3650 1950 50  0001 C CNN
 F 3 "" H 3650 1950 50  0001 C CNN
 	1    3650 1950
@@
 F 0 "C26" H 2510 2770 50  0000 L CNN
 F 1 "C_Small" H 2510 2620 50  0000 L CNN
-F 2 "Capacitors_THT:C_Disc_D7.5mm_W5.0mm_P7.50mm" H 2500 2700 50  0001 C CNN
+F 2 "PA:C_Disc_SMD" H 2500 2700 50  0001 C CNN
 F 3 "" H 2500 2700 50  0001 C CNN
 	1    2500 2700
@@
 F 0 "C28" H 3060 2820 50  0000 L CNN
 F 1 "C_Small" H 3060 2670 50  0000 L CNN
-F 2 "Capacitors_THT:C_Disc_D7.5mm_W5.0mm_P7.50mm" H 3050 2750 50  0001 C CNN
+F 2 "PA:C_Disc_SMD" H 3050 2750 50  0001 C CNN
 F 3 "" H 3050 2750 50  0001 C CNN
 	1    3050 2750
@@
 F 0 "C30" H 3660 2820 50  0000 L CNN
 F 1 "C_Small" H 3660 2670 50  0000 L CNN
-F 2 "Capacitors_THT:C_Disc_D7.5mm_W5.0mm_P7.50mm" H 3650 2750 50  0001 C CNN
+F 2 "PA:C_Disc_SMD" H 3650 2750 50  0001 C CNN
 F 3 "" H 3650 2750 50  0001 C CNN
 	1    3650 2750
@@
 F 0 "C27" H 2510 3620 50  0000 L CNN
 F 1 "C_Small" H 2510 3470 50  0000 L CNN
-F 2 "Capacitors_THT:C_Disc_D7.5mm_W5.0mm_P7.50mm" H 2500 3550 50  0001 C CNN
+F 2 "PA:C_Disc_SMD" H 2500 3550 50  0001 C CNN
 F 3 "" H 2500 3550 50  0001 C CNN
 	1    2500 3550
@@
 F 0 "C29" H 3060 3670 50  0000 L CNN
 F 1 "C_Small" H 3060 3520 50  0000 L CNN
-F 2 "Capacitors_THT:C_Disc_D7.5mm_W5.0mm_P7.50mm" H 3050 3600 50  0001 C CNN
+F 2 "PA:C_Disc_SMD" H 3050 3600 50  0001 C CNN
 F 3 "" H 3050 3600 50  0001 C CNN
 	1    3050 3600
@@
 F 0 "C31" H 3660 3670 50  0000 L CNN
 F 1 "C_Small" H 3660 3520 50  0000 L CNN
-F 2 "Capacitors_THT:C_Disc_D7.5mm_W5.0mm_P7.50mm" H 3650 3600 50  0001 C CNN
+F 2 "PA:C_Disc_SMD" H 3650 3600 50  0001 C CNN
 F 3 "" H 3650 3600 50  0001 C CNN
 	1    3650 3600
@@
 F 0 "C32" H 2510 4470 50  0000 L CNN
 F 1 "C_Small" H 2510 4320 50  0000 L CNN
-F 2 "Capacitors_THT:C_Disc_D7.5mm_W5.0mm_P7.50mm" H 2500 4400 50  0001 C CNN
+F 2 "PA:C_Disc_SMD" H 2500 4400 50  0001 C CNN
 F 3 "" H 2500 4400 50  0001 C CNN
 	1    2500 4400
@@
 F 0 "C34" H 3060 4520 50  0000 L CNN
 F 1 "C_Small" H 3060 4370 50  0000 L CNN
-F 2 "Capacitors_THT:C_Disc_D7.5mm_W5.0mm_P7.50mm" H 3050 4450 50  0001 C CNN
+F 2 "PA:C_Disc_SMD" H 3050 4450 50  0001 C CNN
 F 3 "" H 3050 4450 50  0001 C CNN
 	1    3050 4450
@@
 F 0 "C36" H 3660 4520 50  0000 L CNN
 F 1 "C_Small" H 3660 4370 50  0000 L CNN
-F 2 "Capacitors_THT:C_Disc_D7.5mm_W5.0mm_P7.50mm" H 3650 4450 50  0001 C CNN
+F 2 "PA:C_Disc_SMD" H 3650 4450 50  0001 C CNN
 F 3 "" H 3650 4450 50  0001 C CNN
 	1    3650 4450
@@
 F 0 "C33" H 2510 5320 50  0000 L CNN
 F 1 "C_Small" H 2510 5170 50  0000 L CNN
-F 2 "Capacitors_THT:C_Disc_D7.5mm_W5.0mm_P7.50mm" H 2500 5250 50  0001 C CNN
+F 2 "PA:C_Disc_SMD" H 2500 5250 50  0001 C CNN
 F 3 "" H 2500 5250 50  0001 C CNN
 	1    2500 5250
@@
 F 0 "C35" H 3060 5370 50  0000 L CNN
 F 1 "C_Small" H 3060 5220 50  0000 L CNN
-F 2 "Capacitors_THT:C_Disc_D7.5mm_W5.0mm_P7.50mm" H 3050 5300 50  0001 C CNN
+F 2 "PA:C_Disc_SMD" H 3050 5300 50  0001 C CNN
 F 3 "" H 3050 5300 50  0001 C CNN
 	1    3050 5300
@@
 F 0 "C37" H 3660 5370 50  0000 L CNN
 F 1 "C_Small" H 3660 5220 50  0000 L CNN
-F 2 "Capacitors_THT:C_Disc_D7.5mm_W5.0mm_P7.50mm" H 3650 5300 50  0001 C CNN
+F 2 "PA:C_Disc_SMD" H 3650 5300 50  0001 C CNN
 F 3 "" H 3650 5300 50  0001 C CNN
 	1    3650 5300

Commit message: Some more comitization
Parts:
- added J29, J30: Conn_01x01, Connectors:1pin, symbol Conn_01x01
Connections:
- net GND: now also J29.1 (Pin_1), J30.1 (Pin_1)
Changed lines of the file:
@@
 $EndComp
 $Comp
-L GND #PWR049
+L GND #PWR56
 U 1 1 5C655510
 P 2500 2100
-F 0 "#PWR049" H 2500 1850 50  0001 C CNN
+F 0 "#PWR56" H 2500 1850 50  0001 C CNN
 F 1 "GND" H 2500 1950 50  0000 C CNN
 F 2 "" H 2500 2100 50  0001 C CNN
@@
 	3050 1750 3050 1850
 $Comp
-L GND #PWR050
+L GND #PWR61
 U 1 1 5C6555C6
 P 3050 2100
-F 0 "#PWR050" H 3050 1850 50  0001 C CNN
+F 0 "#PWR61" H 3050 1850 50  0001 C CNN
 F 1 "GND" H 3050 1950 50  0000 C CNN
 F 2 "" H 3050 2100 50  0001 C CNN
@@
 $EndComp
 $Comp
-L GND #PWR051
+L GND #PWR66
 U 1 1 5C65564F
 P 3650 2100
-F 0 "#PWR051" H 3650 1850 50  0001 C CNN
+F 0 "#PWR66" H 3650 1850 50  0001 C CNN
 F 1 "GND" H 3650 1950 50  0000 C CNN
 F 2 "" H 3650 2100 50  0001 C CNN
@@
 $EndComp
 $Comp
-L GND #PWR052
+L GND #PWR57
 U 1 1 5C655E84
 P 2500 2900
-F 0 "#PWR052" H 2500 2650 50  0001 C CNN
+F 0 "#PWR57" H 2500 2650 50  0001 C CNN
 F 1 "GND" H 2500 2750 50  0000 C CNN
 F 2 "" H 2500 2900 50  0001 C CNN
@@
 	3050 2550 3050 2650
 $Comp
-L GND #PWR053
+L GND #PWR62
 U 1 1 5C655E9C
 P 3050 2900
-F 0 "#PWR053" H 3050 2650 50  0001 C CNN
+F 0 "#PWR62" H 3050 2650 50  0001 C CNN
 F 1 "GND" H 3050 2750 50  0000 C CNN
 F 2 "" H 3050 2900 50  0001 C CNN
@@
 $EndComp
 $Comp
-L GND #PWR054
+L GND #PWR67
 U 1 1 5C655EB0
 P 3650 2900
-F 0 "#PWR054" H 3650 2650 50  0001 C CNN
+F 0 "#PWR67" H 3650 2650 50  0001 C CNN
 F 1 "GND" H 3650 2750 50  0000 C CNN
 F 2 "" H 3650 2900 50  0001 C CNN
@@
 $EndComp
 $Comp
-L GND #PWR055
+L GND #PWR58
 U 1 1 5C656083
 P 2500 3750
-F 0 "#PWR055" H 2500 3500 50  0001 C CNN
+F 0 "#PWR58" H 2500 3500 50  0001 C CNN
 F 1 "GND" H 2500 3600 50  0000 C CNN
 F 2 "" H 2500 3750 50  0001 C CNN
@@
 	3050 3400 3050 3500
 $Comp
-L GND #PWR056
+L GND #PWR63
 U 1 1 5C65609B
 P 3050 3750
-F 0 "#PWR056" H 3050 3500 50  0001 C CNN
+F 0 "#PWR63" H 3050 3500 50  0001 C CNN
 F 1 "GND" H 3050 3600 50  0000 C CNN
 F 2 "" H 3050 3750 50  0001 C CNN
@@
 $EndComp
 $Comp
-L GND #PWR057
+L GND #PWR68
 U 1 1 5C6560AF
 P 3650 3750
-F 0 "#PWR057" H 3650 3500 50  0001 C CNN
+F 0 "#PWR68" H 3650 3500 50  0001 C CNN
 F 1 "GND" H 3650 3600 50  0000 C CNN
 F 2 "" H 3650 3750 50  0001 C CNN
@@
 $EndComp
 $Comp
-L GND #PWR058
+L GND #PWR59
 U 1 1 5C656528
 P 2500 4600
-F 0 "#PWR058" H 2500 4350 50  0001 C CNN
+F 0 "#PWR59" H 2500 4350 50  0001 C CNN
 F 1 "GND" H 2500 4450 50  0000 C CNN
 F 2 "" H 2500 4600 50  0001 C CNN
@@
 	3050 4250 3050 4350
 $Comp
-L GND #PWR059
+L GND #PWR64
 U 1 1 5C656540
 P 3050 4600
-F 0 "#PWR059" H 3050 4350 50  0001 C CNN
+F 0 "#PWR64" H 3050 4350 50  0001 C CNN
 F 1 "GND" H 3050 4450 50  0000 C CNN
 F 2 "" H 3050 4600 50  0001 C CNN
@@
 $EndComp
 $Comp
-L GND #PWR060
+L GND #PWR69
 U 1 1 5C656554
 P 3650 4600
-F 0 "#PWR060" H 3650 4350 50  0001 C CNN
+F 0 "#PWR69" H 3650 4350 50  0001 C CNN
 F 1 "GND" H 3650 4450 50  0000 C CNN
 F 2 "" H 3650 4600 50  0001 C CNN
@@
 $EndComp
 $Comp
-L GND #PWR061
+L GND #PWR60
 U 1 1 5C65665B
 P 2500 5450
-F 0 "#PWR061" H 2500 5200 50  0001 C CNN
+F 0 "#PWR60" H 2500 5200 50  0001 C CNN
 F 1 "GND" H 2500 5300 50  0000 C CNN
 F 2 "" H 2500 5450 50  0001 C CNN
@@
 	3050 5100 3050 5200
 $Comp
-L GND #PWR062
+L GND #PWR65
 U 1 1 5C656673
 P 3050 5450
-F 0 "#PWR062" H 3050 5200 50  0001 C CNN
+F 0 "#PWR65" H 3050 5200 50  0001 C CNN
 F 1 "GND" H 3050 5300 50  0000 C CNN
 F 2 "" H 3050 5450 50  0001 C CNN
@@
 $EndComp
 $Comp
-L GND #PWR063
+L GND #PWR70
 U 1 1 5C656687
 P 3650 5450
-F 0 "#PWR063" H 3650 5200 50  0001 C CNN
+F 0 "#PWR70" H 3650 5200 50  0001 C CNN
 F 1 "GND" H 3650 5300 50  0000 C CNN
 F 2 "" H 3650 5450 50  0001 C CNN
@@
 $EndComp
 $Comp
-L GND #PWR064
+L GND #PWR49
 U 1 1 5C656E4F
 P 1150 1700
-F 0 "#PWR064" H 1150 1450 50  0001 C CNN
+F 0 "#PWR49" H 1150 1450 50  0001 C CNN
 F 1 "GND" H 1150 1550 50  0000 C CNN
 F 2 "" H 1150 1700 50  0001 C CNN
@@
 	1150 1700 1000 1700
 $Comp
-L GND #PWR065
+L GND #PWR50
 U 1 1 5C656F3E
 P 1150 2000
-F 0 "#PWR065" H 1150 1750 50  0001 C CNN
+F 0 "#PWR50" H 1150 1750 50  0001 C CNN
 F 1 "GND" H 1150 1850 50  0000 C CNN
 F 2 "" H 1150 2000 50  0001 C CNN
@@
 	1150 2000 1000 2000
 $Comp
-L GND #PWR066
+L GND #PWR51
 U 1 1 5C65702E
 P 1200 2350
-F 0 "#PWR066" H 1200 2100 50  0001 C CNN
+F 0 "#PWR51" H 1200 2100 50  0001 C CNN
 F 1 "GND" H 1200 2200 50  0000 C CNN
 F 2 "" H 1200 2350 50  0001 C CNN
@@
 	1200 2350 1000 2350
 $Comp
-L GND #PWR067
+L GND #PWR52
 U 1 1 5C65711F
 P 1200 2650
-F 0 "#PWR067" H 1200 2400 50  0001 C CNN
+F 0 "#PWR52" H 1200 2400 50  0001 C CNN
 F 1 "GND" H 1200 2500 50  0000 C CNN
 F 2 "" H 1200 2650 50  0001 C CNN
@@
 $EndComp
 $Comp
-L GND #PWR068
+L GND #PWR53
 U 1 1 5C658518
 P 1200 2950
-F 0 "#PWR068" H 1200 2700 50  0001 C CNN
+F 0 "#PWR53" H 1200 2700 50  0001 C CNN
 F 1 "GND" H 1200 2800 50  0000 C CNN
 F 2 "" H 1200 2950 50  0001 C CNN
@@
 Wire Wire Line
 	1200 2950 1000 2950
+$Comp
+L Conn_01x01 J29
+U 1 1 5C664D5E
+P 800 3250
+F 0 "J29" H 800 3350 50  0000 C CNN
+F 1 "Conn_01x01" H 800 3150 50  0000 C CNN
+F 2 "Connectors:1pin" H 800 3250 50  0001 C CNN
+F 3 "" H 800 3250 50  0001 C CNN
+	1    800  3250
+	-1   0    0    1
+$EndComp
+$Comp
+L GND #PWR54
+U 1 1 5C664D64
+P 1200 3250
+F 0 "#PWR54" H 1200 3000 50  0001 C CNN
+F 1 "GND" H 1200 3100 50  0000 C CNN
+F 2 "" H 1200 3250 50  0001 C CNN
+F 3 "" H 1200 3250 50  0001 C CNN
+	1    1200 3250
+	0    -1   -1   0
+$EndComp
+Wire Wire Line
+	1200 3250 1000 3250
+$Comp
+L Conn_01x01 J30
+U 1 1 5C664D6B
+P 800 3550
+F 0 "J30" H 800 3650 50  0000 C CNN
+F 1 "Conn_01x01" H 800 3450 50  0000 C CNN
+F 2 "Connectors:1pin" H 800 3550 50  0001 C CNN
+F 3 "" H 800 3550 50  0001 C CNN
+	1    800  3550
+	-1   0    0    1
+$EndComp
+$Comp
+L GND #PWR55
+U 1 1 5C664D71
+P 1200 3550
+F 0 "#PWR55" H 1200 3300 50  0001 C CNN
+F 1 "GND" H 1200 3400 50  0000 C CNN
+F 2 "" H 1200 3550 50  0001 C CNN
+F 3 "" H 1200 3550 50  0001 C CNN
+	1    1200 3550
+	0    -1   -1   0
+$EndComp
+Wire Wire Line
+	1200 3550 1000 3550
 $EndSCHEMATC
