File: Filter/Filter.kicad_pcb (KiCad board)
At the start: 2 copper layers, 100 x 100 mm, 69 parts, among them J1 Conn_Coaxial, J10 Conn_01x02, J11 Conn_01x08, J2 Conn_01x02, J3 Conn_Coaxial, J4 Conn_01x02, J5 Conn_01x02, J6 Conn_01x01, J7 Conn_01x01, J8 Conn_01x01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

Commit message: Added some extra protection and fixed labels on Filter
Parts:
- added C25: C, Capacitors_THT:C_Disc_D5.0mm_W2.5mm_P2.50mm, F.Cu at (51.3, 98.3)
- added C26: C, Capacitors_THT:C_Disc_D5.0mm_W2.5mm_P2.50mm, F.Cu at (51.3, 101.1)
- added C33: C, Capacitors_THT:C_Disc_D5.0mm_W2.5mm_P2.50mm, F.Cu at (51.2, 104.0)
- added C34: C, Capacitors_THT:C_Disc_D5.0mm_W2.5mm_P2.50mm, F.Cu at (51.2, 106.6)
- added C35: C, Capacitors_THT:C_Disc_D5.0mm_W2.5mm_P2.50mm, F.Cu at (51.1, 109.3)
- added C36: C, Capacitors_THT:C_Disc_D5.0mm_W2.5mm_P2.50mm, F.Cu at (51.2, 112.0)
- added C37: 100 nF, Capacitors_THT:C_Disc_D5.0mm_W2.5mm_P2.50mm, F.Cu at (52.6, 122.5)
- R3, R4: value 10k -> 100k
Routing:
- net +12V: track 179.3 -> 188.8 mm
- net Net-(C25-Pad1): track 16.4 -> 23.5 mm
- net Net-(C34-Pad1): track 16.4 -> 22.9 mm
- net Net-(C26-Pad1): track 16.4 -> 22.6 mm
- net Net-(C33-Pad1): track 16.4 -> 21.8 mm
- net Net-(C35-Pad1): track 17.4 -> 22.1 mm
- net Net-(C36-Pad1): track 18.1 -> 20.2 mm

Commit message: Added tandem match to sense power to filter board
Parts:
- added C38: 100 nF, Capacitors_THT:C_Disc_D5.0mm_W2.5mm_P2.50mm, F.Cu at (48.5, 80.5)
- added C39: 100 nF, Capacitors_THT:C_Disc_D5.0mm_W2.5mm_P2.50mm, F.Cu at (44.5, 64.3)
- added D4: 1N5711, Diodes_THT:D_DO-35_SOD27_P7.62mm_Horizontal, F.Cu at (45.2, 76.2)
- added D5: 1N5711, Diodes_THT:D_DO-35_SOD27_P7.62mm_Horizontal, F.Cu at (42.2, 56.9)
- added J16: Conn_01x01, Connectors:1pin, F.Cu at (53.8, 56.1)
- added J17: Conn_01x01, Connectors:1pin, F.Cu at (66.5, 71.1)
- added J18: Conn_01x01, Connectors:1pin, F.Cu at (61.0, 52.1)
- added J19: Conn_01x01, Connectors:1pin, F.Cu at (61.0, 60.7)
- added J20: Conn_01x01, Connectors:1pin, F.Cu at (59.7, 67.1)
- added J21: Conn_01x01, Connectors:1pin, F.Cu at (60.2, 75.9)
- added J22: Conn_01x01, Connectors:1pin, F.Cu at (67.6, 56.1)
- added J23: Conn_01x01, Connectors:1pin, F.Cu at (53.1, 70.6)
- added R11: 10k, Resistors_THT:R_Axial_DIN0207_L6.3mm_D2.5mm_P7.62mm_Horizontal, F.Cu at (42.4, 53.8)
- added R12: 10k, Resistors_THT:R_Axial_DIN0207_L6.3mm_D2.5mm_P7.62mm_Horizontal, F.Cu at (50.0, 50.8)
- added R5: 10k, Resistors_THT:R_Axial_DIN0207_L6.3mm_D2.5mm_P7.62mm_Horizontal, F.Cu at (42.7, 68.6)
- added R6: 10k, Resistors_THT:R_Axial_DIN0207_L6.3mm_D2.5mm_P7.62mm_Horizontal, F.Cu at (51.1, 88.1)
- added R7: 51R, Resistors_THT:R_Axial_DIN0309_L9.0mm_D3.2mm_P12.70mm_Horizontal, F.Cu at (48.5, 63.8)
- added R8: 51R, Resistors_THT:R_Axial_DIN0309_L9.0mm_D3.2mm_P12.70mm_Horizontal, F.Cu at (55.4, 60.5)
- J10: value Conn_01x02 -> Conn_01x04; footprint Connectors_Terminal_Blocks:TerminalBlock_bornier-2_P5.08mm -> Connectors_Molex:Molex_KK-6410-04_04x2.54mm_Straight
- moved J2 34.0 mm to (56.9, 45.5)
- moved R3 33.2 mm to (66.2, 98.6), turned to 90 degrees
- moved R4 30.4 mm to (56.9, 91.9), turned to 180 degrees
- moved C20 30.1 mm to (52.1, 76.2)
- moved R1 28.2 mm to (66.8, 80.0)
- moved R2 27.6 mm to (51.6, 84.3)
- moved C22 27.4 mm to (63.4, 87.8), turned to 0 degrees
- moved D1 26.7 mm to (63.2, 98.4), turned to 90 degrees
- moved D2 22.1 mm to (60.2, 90.9), turned to 270 degrees
- moved C24 22.0 mm to (64.9, 101.6)
- moved D3 21.9 mm to (57.1, 95.2)
- moved J10 13.7 mm to (44.5, 85.9), turned to 270 degrees
- moved J1 6.32 mm to (68.3, 35.8)
- moved J11 0.60 mm to (45.0, 99.3)
Connections:
- J10 pad 1: Net-(C22-Pad1) -> Net-(C39-Pad1)
- J10 pad 2: GND -> Net-(C38-Pad1)
- RLY1 pad 2: INRF -> Net-(J22-Pad1)
- RLY2 pad 2: INRF -> Net-(J22-Pad1)
- RLY3 pad 2: INRF -> Net-(J22-Pad1)
- RLY4 pad 2: INRF -> Net-(J22-Pad1)
- RLY5 pad 2: INRF -> Net-(J22-Pad1)
- RLY6 pad 2: INRF -> Net-(J22-Pad1)
Routing:
- net GND: track 0.72 -> 160.5 mm, vias 0 -> 69
- net Net-(J22-Pad1): track 0.00 -> 110.4 mm
- net INRF: track 128.4 -> 85.8 mm
- net Net-(C39-Pad1): track 0.00 -> 42.3 mm
- net Net-(D4-Pad2): track 0.00 -> 34.3 mm
- net Net-(D5-Pad2): track 0.00 -> 25.6 mm
- net Net-(C38-Pad1): track 0.00 -> 24.3 mm
- net Net-(D4-Pad1): track 0.00 -> 8.05 mm
- net Net-(C20-Pad1): track 17.6 -> 24.1 mm
- net Net-(D5-Pad1): track 0.00 -> 3.15 mm
- net Net-(C25-Pad1): track 23.5 -> 21.8 mm
- net Net-(C26-Pad1): track 22.6 -> 21.1 mm
- net Net-(C33-Pad1): track 21.8 -> 20.5 mm
- net Net-(C24-Pad1): track 16.4 -> 15.4 mm
- net Net-(C35-Pad1): track 22.1 -> 22.7 mm
Other:
- board text removed: "DIG"

Commit message: Moved series resistor closer to common drain amplifier to prevent oscillation
Parts:
- added C40: C_Small, FilterD:C_Disc_SMD, F.Cu at (110.0, 119.9)
- added C41: C_Small, FilterD:C_Disc_SMD, F.Cu at (110.5, 54.1)
- added C42: C_Small, FilterD:C_Disc_SMD, F.Cu at (110.2, 70.1)
- added C43: C_Small, FilterD:C_Disc_SMD, F.Cu at (110.0, 87.6)
- added C44: C_Small, FilterD:C_Disc_SMD, F.Cu at (110.2, 103.9)
- added C45: C_Small, FilterD:C_Disc_SMD, F.Cu at (110.5, 128.8)
- added C46: C_Small, FilterD:C_Disc_SMD, F.Cu at (128.3, 54.1)
- added C47: C_Small, FilterD:C_Disc_SMD, F.Cu at (129.0, 119.9)
- added C48: C_Small, FilterD:C_Disc_SMD, F.Cu at (128.3, 70.4)
- added C49: C_Small, FilterD:C_Disc_SMD, F.Cu at (128.3, 87.4)
- added C50: C_Small, FilterD:C_Disc_SMD, F.Cu at (129.3, 103.9)
- added C51: C_Small, FilterD:C_Disc_SMD, F.Cu at (127.8, 128.5)
- L1, L10, L11, L12, L2, L3, L4, L5, L6, L7, L8, L9: footprint Inductors_THT:L_Toroid_Vertical_L13.0mm_W6.5mm_P5.60mm -> FilterD:L_Toroid_Vertical_L13.0mm_W6.5mm_P5.60mm_mod
- moved C6 12.3 mm to (96.8, 138.4), turned to 90 degrees
- moved C8 9.96 mm to (115.3, 62.0), turned to 270 degrees
- moved C9 9.90 mm to (115.3, 78.5), turned to 270 degrees
- moved C7 9.52 mm to (115.6, 46.7), turned to 270 degrees
- moved C10 8.62 mm to (115.6, 94.7), turned to 270 degrees
- moved C18 7.97 mm to (133.3, 130.6), turned to 90 degrees
- moved C11 7.81 mm to (116.1, 111.3), turned to 270 degrees
- moved L12 6.48 mm to (122.2, 136.4)
- moved L2 5.60 mm to (103.4, 63.0)
- moved L6 5.54 mm to (103.9, 136.4)
- moved L1 5.32 mm to (103.9, 47.2)
- moved L7 5.22 mm to (121.4, 47.5)
- moved L8 5.14 mm to (121.9, 63.0)
- moved L10 4.93 mm to (122.4, 95.0)
- moved C12 4.74 mm to (115.3, 138.4)
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Routing:
- net Net-(C10-Pad1): track 15.7 -> 33.0 mm
- net Net-(C12-Pad1): track 15.8 -> 30.5 mm
- net Net-(C11-Pad1): track 17.5 -> 31.6 mm
- net Net-(C42-Pad1): track 15.7 -> 29.0 mm
- net Net-(C43-Pad1): track 17.2 -> 29.8 mm
- net Net-(C45-Pad2): track 15.8 -> 27.7 mm
- net Net-(C41-Pad1): track 16.0 -> 26.6 mm
- net Net-(C16-Pad1): track 51.4 -> 60.4 mm
- net Net-(C3-Pad1): track 17.0 -> 24.6 mm
- net Net-(C18-Pad1): track 52.3 -> 59.6 mm
- net Net-(C1-Pad1): track 20.1 -> 26.5 mm
- net Net-(C40-Pad2): track 17.1 -> 23.5 mm
- net Net-(C4-Pad1): track 16.5 -> 22.8 mm
- net Net-(C17-Pad1): track 50.8 -> 56.8 mm
- net Net-(C2-Pad1): track 20.0 -> 25.7 mm
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